File: Electrical/ESC-BLDC-FORMULA1-V1_2/bldc-75v.kicad_pcb (KiCad board)
At the start: 4 copper layers, 140 x 105.3 mm, 122 parts, among them J10 CAN, J5 Battery (anti-spark in cable), J6 Motor-Phases, J7 Throttle, J8 Hall, J9 UART, Q1 CSD19532Q5B, Q2 CSD19532Q5B, Q3 CSD19532Q5B, Q4 CSD19532Q5B, Q5 CSD19532Q5B, Q6 CSD19532Q5B, U1 DRV8353RSRGZT, U2 NUCLEO-G474RE, U3 TPD4S010DQAR, U4 LM5164DDA, U5 TJA1051T/3

Commit message: ESC: final ordered V1.2, handoff notes for Claude Code, JLC tools
- Board/schematic/JLC files exactly as ordered at JLCPCB (generated
  2026-09-30): motor temperature input on J8 pin 6 -> PA7, GND via for the
  C67 island, C31 via moved, R73 label, J8/J9/J10 1.0 mm holes
- CLAUDE.md: status, hardware facts, motor data, car-level decisions,
  firmware decisions and to-do list, release checklist, gotchas
- tools/: gen_jlc.py + lcsc_map.py (reproduce the ordered BOM/CPL byte for
  byte), overlay.py (JLC footprint rotation check), dfm_checks.py
- README: 6-pin J8, PA7 motor temperature, order status, tools
- firmware/README: bring up at 20-24 V (LM5164 EN/UVLO turns on at 18 V)

Co-Authored-By: Claude Opus 5.5 <noreply@anthropic.com>
Parts:
- added C67: 100nF, Capacitor_SMD:C_0603_1608Metric, F.Cu at (177.4, 66.6)
- added R73: 2.2k, Resistor_SMD:R_0603_1608Metric, F.Cu at (173.6, 66.6)
- added R74: 1k, Resistor_SMD:R_0603_1608Metric, F.Cu at (175.5, 66.6)
- J8: footprint Connector_JST:JST_XH_B5B-XH-A_1x05_P2.50mm_Vertical -> Connector_JST:JST_XH_B6B-XH-A_1x06_P2.50mm_Vertical
Connections:
- U2 pad CN10_15: unconnected-(U2B-PA7-PadCN10_15) -> /MOT_TEMP_ADC
Routing:
- net /MOT_TEMP: track 0.00 -> 50.1 mm
- net /MOT_TEMP_ADC: track 0.00 -> 10.6 mm, vias 0 -> 1
- net +3V3: track 272.7 -> 275.8 mm, vias 8 -> 9
- net GND: track 77.3 -> 77.4 mm, vias 99 -> 100
Other:
- board text added: "T"
