File: Electrical/ESC-BLDC-FORMULA1-V1_2/bldc-75v.kicad_sch (KiCad schematic)
At the start: 118 parts, among them J10 CAN, J5 Battery (anti-spark in cable), J6 Motor-Phases, J7 Throttle, J8 Hall, J9 UART, Q1 CSD19532Q5B, Q2 CSD19532Q5B, Q3 CSD19532Q5B, Q4 CSD19532Q5B, Q5 CSD19532Q5B, Q6 CSD19532Q5B, U1 DRV8353RSRGZT, U2 NUCLEO-G474RE, U3 TPD4S010DQAR, U4 LM5164DDA, U5 TJA1051T/3

Commit message: ESC: final ordered V1.2, handoff notes for Claude Code, JLC tools
- Board/schematic/JLC files exactly as ordered at JLCPCB (generated
  2026-09-30): motor temperature input on J8 pin 6 -> PA7, GND via for the
  C67 island, C31 via moved, R73 label, J8/J9/J10 1.0 mm holes
- CLAUDE.md: status, hardware facts, motor data, car-level decisions,
  firmware decisions and to-do list, release checklist, gotchas
- tools/: gen_jlc.py + lcsc_map.py (reproduce the ordered BOM/CPL byte for
  byte), overlay.py (JLC footprint rotation check), dfm_checks.py
- README: 6-pin J8, PA7 motor temperature, order status, tools
- firmware/README: bring up at 20-24 V (LM5164 EN/UVLO turns on at 18 V)

Co-Authored-By: Claude Opus 5.5 <noreply@anthropic.com>
Parts:
- added C67: 100nF, Capacitor_SMD:C_0603_1608Metric, symbol Device:C_Small
- added R73: 2.2k, Resistor_SMD:R_0603_1608Metric, symbol Device:R
- added R74: 1k, Resistor_SMD:R_0603_1608Metric, symbol Device:R
- J8: footprint Connector_JST:JST_XH_B5B-XH-A_1x05_P2.50mm_Vertical -> Connector_JST:JST_XH_B6B-XH-A_1x06_P2.50mm_Vertical; symbol Connector:Conn_01x05_Pin -> Connector:Conn_01x06_Pin; LCSC C378947 -> C144397
Connections:
- net +3V3: now also R73.1
- net GND: now also C67.2
- net MOT_TEMP_ADC: now reaches U2.CN10_15 (PA7)
- net MOT_TEMP_ADC: now also C67.1, R74.2
- new net MOT_TEMP: J8.6 (Pin_6), R73.2, R74.1
- no-connect marks 39 -> 38
Other:
- note added: "Motor temperature (J8 pin 6, white wire) -> PA7 / ADC2_IN4. Sensor type unknown: 2.2k pull-up works for NTC 10k, KTY84, PT1000"
