File: Electrical/ESC-BLDC-FORMULA1-V2_0/bldc-75v.kicad_sch (KiCad schematic)
At the start: 118 parts, among them J10 CAN, J11 Wheel, J12 MOTB, J13 MOTA, J5 Battery (anti-spark in cable), J6 MOTC, J7 Throttle, J8 Hall, J9 UART, Q1 CSD19532Q5B, Q2 CSD19532Q5B, Q3 CSD19532Q5B, Q4 CSD19532Q5B, Q5 CSD19532Q5B, Q6 CSD19532Q5B, U1 DRV8353RSRGZT, U2 NUCLEO-G474RE, U5 TJA1051T/3, U6 TPS562201

Commit message: ESC V2.0: 60 V safe TVS (SMCJ60A), keep DRV8353 low-side current sensing
- D8 SMCJ54A -> SMCJ60A (C224057): the 54 V part starts conducting at 60 V and would
  overheat on a 60 V battery; SMCJ60A breaks down at 66.7 V min, clamps at 96.8 V
- Current sensing stays low-side with the DRV8353 amplifiers (inline INA240 variant
  kept as tools/optional/v2_sch_inline.py, not applied)
- All parts on the battery line checked for 60 V: FETs 100 V, VDRAIN 100 V,
  DRV buck VIN 95 V, VM from the 12 V buck, caps 100 V

Co-Authored-By: Claude Opus 5.5 <noreply@anthropic.com>
Parts:
- D8: value SMCJ54A -> SMCJ60A; LCSC C2943841 -> C224057
Changed lines of the file:
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@@
 			)
 		)
-		(property "Value" "SMCJ54A"
+		(property "Value" "SMCJ60A"
 			(at 358.14 128.27 0)
 			(show_name no)
@@
 			)
 		)
-		(property "Description" "Unidirectional TVS 54V standoff (12S pack 50.4 V), 87 V clamp"
+		(property "Description" "Bus TVS 60 V standoff (breakdown 66.7 V min, clamp 96.8 V): safe with a 60 V battery"
 			(at 355.6 127 0)
 			(hide yes)
@@
 			)
 		)
-		(property "LCSC" "C2943841"
+		(property "LCSC" "C224057"
 			(at 355.6 127 0)
 			(hide yes)

Commit message: ESC V2.0: big THT bus caps again (3x 330 uF 100 V)
C11/C21/C68: 330 uF 100 V 16x25 mm THT (Samyoung NXA C346987, the V1.2 part, 1.65 A
ripple each = ~5 A) instead of SMD 47 uF 10x10 (too little ripple rating). Placed in
the free corners beside the phase cells, outside the Nucleo area; board 110.5 x 90 mm
(x 143-253.5), right corner holes moved. Parity 0, no courtyard overlaps.

Co-Authored-By: Claude Opus 5.5 <noreply@anthropic.com>
Parts:
- C11, C21, C68: value 47uF 100V -> 330uF 100V; footprint Capacitor_SMD:CP_Elec_10x10 -> Capacitor_THT:CP_Radial_D16.0mm_P7.50mm; LCSC C164068 -> C346987
Changed lines of the file:
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@@
 			)
 		)
-		(property "Value" "47uF 100V"
+		(property "Value" "330uF 100V"
 			(at 264.16 148.9709 0)
 			(show_name no)
@@
 			)
 		)
-		(property "Footprint" "Capacitor_SMD:CP_Elec_10x10"
+		(property "Footprint" "Capacitor_THT:CP_Radial_D16.0mm_P7.50mm"
 			(at 261.3152 152.4 0)
 			(hide yes)
@@
 			)
 		)
-		(property "Description" "Polarized capacitor"
+		(property "Description" "Bus bulk cap 330 uF 100 V, 16x25 mm, 1.65 A ripple (Samyoung NXA, as V1.2)"
 			(at 260.35 148.59 0)
 			(hide yes)
@@
 			)
 		)
-		(property "LCSC" "C164068"
+		(property "LCSC" "C346987"
 			(at 261.3152 152.4 0)
 			(hide yes)
@@
 			)
 		)
-		(property "Value" "47uF 100V"
+		(property "Value" "330uF 100V"
 			(at 245.11 148.9709 0)
 			(show_name no)
@@
 			)
 		)
-		(property "Footprint" "Capacitor_SMD:CP_Elec_10x10"
+		(property "Footprint" "Capacitor_THT:CP_Radial_D16.0mm_P7.50mm"
 			(at 242.2652 152.4 0)
 			(hide yes)
@@
 			)
 		)
-		(property "Description" "Polarized capacitor"
+		(property "Description" "Bus bulk cap 330 uF 100 V, 16x25 mm, 1.65 A ripple (Samyoung NXA, as V1.2)"
 			(at 241.3 148.59 0)
 			(hide yes)
@@
 			)
 		)
-		(property "LCSC" "C164068"
+		(property "LCSC" "C346987"
 			(at 242.2652 152.4 0)
 			(hide yes)
@@
 			)
 		)
-		(property "Value" "47uF 100V"
+		(property "Value" "330uF 100V"
 			(at 200.66 102.87 0)
 			(show_name no)
@@
 			)
 		)
-		(property "Footprint" "Capacitor_SMD:CP_Elec_10x10"
+		(property "Footprint" "Capacitor_THT:CP_Radial_D16.0mm_P7.50mm"
 			(at 198.12 101.6 0)
 			(hide yes)
@@
 			)
 		)
-		(property "Description" "Bus bulk cap"
+		(property "Description" "Bus bulk cap 330 uF 100 V, 16x25 mm, 1.65 A ripple (Samyoung NXA, as V1.2)"
 			(at 198.12 101.6 0)
 			(hide yes)
@@
 			)
 		)
-		(property "LCSC" "C164068"
+		(property "LCSC" "C346987"
 			(at 198.12 101.6 0)
 			(hide yes)
